File: pcb_kicad/esp32s3_serial_bridge_pcb/esp32s3_serial_bridge_pcb.kicad_pcb (KiCad board)
At the start: 2 copper layers, 11 parts, among them J1 Conn_01x22_Socket, J2 Conn_01x22_Socket, J3 Conn_01x06_Socket, J4 Conn_01x06_Socket, J5 Conn_01x06_Socket, J6 Barrel_Jack_Switch, U2 R-78C5.0-1.0, U3 ESP32-S3-DevKitC-3rd-party-57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

Commit message: add PCB ESP32S3-Serial-Bridge V1.0 Kerberos
add PCB ESP32S3-Serial-Bridge V1.0 Kerberos
Parts:
- U3: value ESP32-S3-DevKitC-3rd-party-57x28 -> ESP32-S3-DevKitC-3rd-party-5715x2794; footprint PCM_Espressif:ESP32-S3-DevKitC_3rd_party_57x28 -> PCM_Espressif:ESP32-S3-DevKitC_3rd_party_5715x2794
- moved J6 78.9 mm to (109.3, 118.1), turned to 90 degrees
- moved C1 65.2 mm to (109.2, 109.1)
- moved U2 63.0 mm to (111.3, 101.2)
- moved C2 57.0 mm to (117.0, 108.1), turned to 180 degrees
- moved C3 53.6 mm to (119.3, 128.7), turned to -90 degrees
- moved J5 46.6 mm to (165.3, 116.9)
- moved J2 43.8 mm to (123.8, 77.1)
- moved J4 27.1 mm to (165.3, 97.7)
- moved J3 8.54 mm to (165.3, 78.4)
- moved U3 8.32 mm to (125.9, 75.0)
- moved J1 8.09 mm to (155.8, 77.1)
Routing:
- net GND: track 0.00 -> 171.1 mm, vias 0 -> 7
- net +5V: track 0.00 -> 119.9 mm
- net GPIO16_CTS0: track 0.00 -> 49.5 mm, vias 0 -> 2
- net GPIO15_RTS0: track 0.00 -> 44.2 mm, vias 0 -> 2
- net GPIO18_RX1: track 0.00 -> 42.8 mm, vias 0 -> 2
- net GPIO17_TX1: track 0.00 -> 42.7 mm, vias 0 -> 2
- net GPIO20_CTS1: track 0.00 -> 32.3 mm
- net GPIO38_RX2: track 0.00 -> 29.3 mm
- net GPIO35_RTS2: track 0.00 -> 26.8 mm
- net GPIO19_RTS1: track 0.00 -> 26.3 mm
- net GPIO37_TX2: track 0.00 -> 24.2 mm, vias 0 -> 1
- net +12V: track 0.00 -> 20.1 mm
- net GPIO36_CTS2: track 0.00 -> 19.1 mm, vias 0 -> 1
- net GPIO43_TX0: track 0.00 -> 13.4 mm
- net GPIO1_RX0: track 0.00 -> 13.3 mm
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- added copper zone on B.Cu, net GND
- added copper zone on F.Cu, net GND
Other:
- board outline added: 65 x 59 mm
- board text added: "ESP32S3-Serial-Bridge 260128 V1.0 Kerberos takurx"

Commit message: PCBもCTS: GPIO20 -> 10, RTS: GPIO19 -> 9 に変更
PCBもCTS: GPIO20 -> 10, RTS: GPIO19 -> 9 に変更
Connections:
- J1 pad 19: GPIO20_CTS1 -> GPIO20
- J1 pad 20: GPIO19_RTS1 -> GPIO19
- J2 pad 15: GPIO9 -> GPIO9_RTS1
- J2 pad 16: GPIO10 -> GPIO10_CTS1
- J4 pad 1: GPIO20_CTS1 -> GPIO10_CTS1
- J4 pad 5: GPIO19_RTS1 -> GPIO9_RTS1
- U3 pad 15: GPIO9 -> GPIO9_RTS1
- U3 pad 16: GPIO10 -> GPIO10_CTS1
- U3 pad 25: GPIO19_RTS1 -> GPIO19
- U3 pad 26: GPIO20_CTS1 -> GPIO20
Routing:
- net GPIO10_CTS1: track 0.00 -> 48.7 mm, vias 0 -> 1
- net GPIO9_RTS1: track 0.00 -> 43.5 mm, vias 0 -> 1
- net GPIO20_CTS1: track 32.3 -> 0.00 mm
- net GPIO19_RTS1: track 26.3 -> 0.00 mm
- net GPIO9: track 3.48 -> 0.00 mm
- net GPIO10: track 3.48 -> 0.00 mm
- net GPIO20: track 0.00 -> 3.27 mm
- net GPIO19: track 0.00 -> 3.27 mm
Other:
- board text added: "ESP32S3-Serial-Bridge 260225 V1.1 Kerberos takurx"
- board text removed: "ESP32S3-Serial-Bridge 260128 V1.0 Kerberos takurx"
Changed lines of the file:
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@@
 	(title_block
 		(title "ESP32S3-Serial-Bridge, Kerberos")
-		(date "2026-01-28")
-		(rev "V1.0")
+		(date "2026-02-25")
+		(rev "V1.1")
 		(company "takurx")
+		(comment 1 "CTS: GPIO20 -> 10, RTS: GPIO19 -> 9 に変更")
 	)
 	(layers
@@
 	(net 2 "GND")
 	(net 3 "+5V")
-	(net 4 "GPIO19_RTS1")
+	(net 4 "GPIO20")
 	(net 5 "GPIO36_CTS2")
 	(net 6 "GPIO37_TX2")
 	(net 7 "GPIO38_RX2")
 	(net 8 "GPIO1_RX0")
-	(net 9 "GPIO20_CTS1")
+	(net 9 "GPIO19")
 	(net 10 "GPIO35_RTS2")
 	(net 11 "GPIO43_TX0")
@@
 	(net 30 "GPIO12")
 	(net 31 "/GPIO7")
-	(net 32 "GPIO10")
+	(net 32 "GPIO10_CTS1")
 	(net 33 "GPIO6")
 	(net 34 "GPIO46")
@@
 	(net 40 "GPIO13")
 	(net 41 "RST")
-	(net 42 "GPIO9")
+	(net 42 "GPIO9_RTS1")
 	(footprint "Capacitor_SMD:C_2220_5750Metric_Pad1.97x5.40mm_HandSolder"
 		(layer "F.Cu")
@@
 			(layers "*.Cu" "*.Mask")
 			(remove_unused_layers no)
-			(net 9 "GPIO20_CTS1")
+			(net 4 "GPIO20")
 			(pinfunction "Pin_19")
 			(pintype "passive")
@@
 			(layers "*.Cu" "*.Mask")
 			(remove_unused_layers no)
-			(net 4 "GPIO19_RTS1")
+			(net 9 "GPIO19")
 			(pinfunction "Pin_20")
 			(pintype "passive")
@@
 			(layers "*.Cu" "*.Mask")
 			(remove_unused_layers no)
-			(net 9 "GPIO20_CTS1")
+			(net 32 "GPIO10_CTS1")
 			(pinfunction "Pin_1")
 			(pintype "passive")
@@
 			(layers "*.Cu" "*.Mask")
 			(remove_unused_layers no)
-			(net 4 "GPIO19_RTS1")
+			(net 42 "GPIO9_RTS1")
 			(pinfunction "Pin_5")
 			(pintype "passive")
@@
 			(layers "*.Cu" "*.Mask")
 			(remove_unused_layers no)
-			(net 42 "GPIO9")
+			(net 42 "GPIO9_RTS1")
 			(pinfunction "Pin_15")
 			(pintype "passive")
@@
 			(layers "*.Cu" "*.Mask")
 			(remove_unused_layers no)
-			(net 32 "GPIO10")
+			(net 32 "GPIO10_CTS1")
 			(pinfunction "Pin_16")
 			(pintype "passive")
@@
 			(layers "*.Cu" "*.Mask")
 			(remove_unused_layers no)
-			(net 42 "GPIO9")
+			(net 42 "GPIO9_RTS1")
 			(pinfunction "GPIO9/ADC1_CH8")
 			(pintype "bidirectional")
@@
 			(layers "*.Cu" "*.Mask")
 			(remove_unused_layers no)
-			(net 32 "GPIO10")
+			(net 32 "GPIO10_CTS1")
 			(pinfunction "GPIO10/ADC1_CH9")
 			(pintype "bidirectional")
@@
 			(layers "*.Cu" "*.Mask")
 			(remove_unused_layers no)
-			(net 4 "GPIO19_RTS1")
+			(net 9 "GPIO19")
 			(pinfunction "GPIO19/USB_D-")
 			(pintype "bidirectional")
@@
 			(layers "*.Cu" "*.Mask")
 			(remove_unused_layers no)
-			(net 9 "GPIO20_CTS1")
+			(net 4 "GPIO20")
 			(pinfunction "GPIO20/USB_D+")
 			(pintype "bidirectional")
@@
 		(layer "Edge.Cuts")
 	)
-	(gr_text "ESP32S3-Serial-Bridge\n260128 V1.0 Kerberos\ntakurx"
+	(gr_text "ESP32S3-Serial-Bridge\n260225 V1.1 Kerberos\ntakurx"
 		(at 104.9 75.8 270)
 		(layer "F.SilkS")
@@
 	)
 	(segment
-		(start 155.8 125.32)
-		(end 152.7518 125.32)
+		(start 152.7518 122.78)
+		(end 152.595 122.6232)
 		(width 1.27)
 		(layer "F.Cu")
@@
 	)
 	(segment
-		(start 152.7518 125.32)
-		(end 152.595 125.1632)
+		(start 155.8 122.78)
+		(end 152.7518 122.78)
 		(width 1.27)
 		(layer "F.Cu")
@@
 	)
 	(segment
-		(start 165.3 107.87)
-		(end 162.538636 107.87)
-		(width 0.4)
-		(layer "B.Cu")
-		(net 4)
-	)
-	(segment
-		(start 159.1 122.02)
-		(end 155.8 125.32)
-		(width 0.4)
-		(layer "B.Cu")
-		(net 4)
-	)
-	(segment
-		(start 162.538636 107.87)
-		(end 159.1 111.308636)
-		(width 0.4)
-		(layer "B.Cu")
-		(net 4)
-	)
-	(segment
-		(start 159.1 111.308636)
-		(end 159.1 122.02)
-		(width 0.4)
-		(layer "B.Cu")
-		(net 4)
-	)
-	(segment
 		(start 155.8 105)
 		(end 160.1 109.3)
@@
 	)
 	(segment
-		(start 152.7518 122.78)
-		(end 152.595 122.6232)
+		(start 155.8 125.32)
+		(end 152.7518 125.32)
 		(width 1.27)
 		(layer "F.Cu")
@@
 	)
 	(segment
-		(start 155.8 122.78)
-		(end 152.7518 122.78)
+		(start 152.7518 125.32)
+		(end 152.595 125.1632)
 		(width 1.27)
 		(layer "F.Cu")
@@
 	)
 	(segment
-		(start 165.3 97.71)
-		(end 158 105.01)
-		(width 0.4)
-		(layer "B.Cu")
-		(net 9)
-	)
-	(segment
-		(start 158 120.58)
-		(end 155.8 122.78)
-		(width 0.4)
-		(layer "B.Cu")
-		(net 9)
-	)
-	(segment
-		(start 158 105.01)
-		(end 158 120.58)
-		(width 0.4)
-		(layer "B.Cu")
-		(net 9)
-	)
-	(segment
 		(start 165.3 127.1)
 		(end 158.8 120.6)
@@
 	)
 	(segment
+		(start 135.4968 115.0032)
+		(end 135.5 115)
+		(width 0.4)
+		(layer "F.Cu")
+		(net 32)
+	)
+	(segment
+		(start 127.195 115.0032)
+		(end 135.4968 115.0032)
+		(width 0.4)
+		(layer "F.Cu")
+		(net 32)
+	)
+	(segment
 		(start 127.195 115.0032)
 		(end 123.9968 115.0032)
@@
 		(net 32)
 	)
+	(via
+		(at 135.5 115)
+		(size 0.6)
+		(drill 0.3)
+		(layers "F.Cu" "B.Cu")
+		(net 32)
+	)
+	(segment
+		(start 146.751 103.749)
+		(end 159.261 103.749)
+		(width 0.4)
+		(layer "B.Cu")
+		(net 32)
+	)
+	(segment
+		(start 159.261 103.749)
+		(end 165.3 97.71)
+		(width 0.4)
+		(layer "B.Cu")
+		(net 32)
+	)
+	(segment
+		(start 135.5 115)
+		(end 146.751 103.749)
+		(width 0.4)
+		(layer "B.Cu")
+		(net 32)
+	)
 	(segment
 		(start 123.9968 89.6032)
@@
 	)
 	(segment
+		(start 141.4632 112.4632)
+		(end 141.5 112.5)
+		(width 0.4)
+		(layer "F.Cu")
+		(net 42)
+	)
+	(segment
+		(start 127.195 112.4632)
+		(end 141.4632 112.4632)
+		(width 0.4)
+		(layer "F.Cu")
+		(net 42)
+	)
+	(segment
 		(start 127.195 112.4632)
 		(end 123.9968 112.4632)
@@
 		(net 42)
 	)
+	(via
+		(at 141.5 112.5)
+		(size 0.6)
+		(drill 0.3)
+		(layers "F.Cu" "B.Cu")
+		(net 42)
+	)
+	(segment
+		(start 162.13 107.87)
+		(end 161.171 108.829)
+		(width 0.4)
+		(layer "B.Cu")
+		(net 42)
+	)
+	(segment
+		(start 161.171 108.829)
+		(end 145.171 108.829)
+		(width 0.4)
+		(layer "B.Cu")
+		(net 42)
+	)
+	(segment
+		(start 165.3 107.87)
+		(end 162.13 107.87)
+		(width 0.4)
+		(layer "B.Cu")
+		(net 42)
+	)
+	(segment
+		(start 145.171 108.829)
+		(end 141.5 112.5)
+		(width 0.4)
+		(layer "B.Cu")
+		(net 42)
+	)
